File: kicad/sensor-node-bl651/power.sch (KiCad schematic (older format))
At the start: 8 parts, among them T1 TPS6031x, U2 DMP2008UFG-7

Commit message: add fuses
Parts:
- removed T1: TPS6031x, Package_SO:MSOP-10_3x3mm_P0.5mm, symbol HH_TexasInstruments:TPS6031x
- added F1: Fuse, Fuse:Fuse_0603_1608Metric, symbol Device:Fuse
- added L1: 4.7µH, Inductor_SMD:L_Taiyo-Yuden_NR-20xx, symbol Device:L
- added P1: TPS61098x, HH_TexasInstruments:TPS61098x, symbol HH_TexasInstruments:TPS61098x
- C2, C4: value 1µF X7R 0603 -> 10µF 0603
- C3: value 1µF X7R 0603 -> 0.1µF 0603
- R3: value 100k 0603 -> 400 0603
Connections:
- net ~SNOOZE is gone; now on net V_BAT: R3.1
- net GND: now also C3.2, C4.2, F1.1, P1.4 (MODE), P1.6 (GND); no longer BT1.2 (-), R3.2
- net V_BAT: now also L1.1
- net V_MAIN: now also C4.1, P1.1 (VMAIN)
- net at C3.1: now also R3.2, P1.3 (VIN)
- new net: L1.2, P1.2 (SW)
- new net: BT1.2 (-), F1.2
- no-connect marks 2 -> 1
Changed lines of the file:
@@
 Comment4 ""
 $EndDescr
-Text HLabel 6550 3650 0    50   Input ~ 0
+$Comp
+L HH_TexasInstruments:TPS61098x P1
+U 1 1 6016D66E
+P 7350 3500
+F 0 "P1" H 7350 3915 50  0000 C CNN
+F 1 "TPS61098x" H 7350 3824 50  0000 C CNN
+F 2 "HH_TexasInstruments:TPS61098x" H 7350 3500 50  0001 C CNN
+F 3 "http://www.ti.com/general/docs/suppproductinfo.tsp?distId=10&gotoUrl=http%3A%2F%2Fwww.ti.com%2Flit%2Fgpn%2Ftps610985" H 7350 3500 50  0001 C CNN
+F 4 "296-48759-6-ND" H 7350 3500 50  0001 C CNN "Digi-Key Part Number"
+F 5 "Texas Instruments" H 7350 3500 50  0001 C CNN "Manufacturer"
+F 6 "TPS61098DSE" H 7350 3500 50  0001 C CNN "Manufacturer Part Number"
+F 7 "IC REG DL BOOST/LNR SYNC 6WSON" H 7350 3500 50  0001 C CNN "Description"
+	1    7350 3500
+	1    0    0    -1
+$EndComp
+$Comp
+L Device:C C2
+U 1 1 6016E335
+P 5350 3500
+F 0 "C2" H 5465 3546 50  0000 L CNN
+F 1 "10µF 0603" H 5465 3455 50  0000 L CNN
+F 2 "Capacitor_SMD:C_0603_1608Metric" H 5388 3350 50  0001 C CNN
+F 3 "~" H 5350 3500 50  0001 C CNN
+	1    5350 3500
+	1    0    0    -1
+$EndComp
+$Comp
+L Device:C C4
+U 1 1 6016E86C
+P 8450 3500
+F 0 "C4" H 8565 3546 50  0000 L CNN
+F 1 "10µF 0603" H 8565 3455 50  0000 L CNN
+F 2 "Capacitor_SMD:C_0603_1608Metric" H 8488 3350 50  0001 C CNN
+F 3 "~" H 8450 3500 50  0001 C CNN
+	1    8450 3500
+	1    0    0    -1
+$EndComp
+Text HLabel 8700 3350 2    50   Input ~ 0
 V_MAIN
+Connection ~ 8450 3350
+Wire Wire Line
+	8450 3350 8700 3350
+Wire Wire Line
+	8000 3650 8050 3650
+$Comp
+L Device:C C3
+U 1 1 60172574
+P 6000 3950
+F 0 "C3" H 6115 3996 50  0000 L CNN
+F 1 "0.1µF 0603" H 6115 3905 50  0000 L CNN
+F 2 "Capacitor_SMD:C_0603_1608Metric" H 6038 3800 50  0001 C CNN
+F 3 "~" H 6000 3950 50  0001 C CNN
+	1    6000 3950
+	1    0    0    -1
+$EndComp
+$Comp
+L Device:L L1
+U 1 1 60173BBD
+P 6350 3350
+F 0 "L1" V 6540 3350 50  0000 C CNN
+F 1 "4.7µH" V 6449 3350 50  0000 C CNN
+F 2 "Inductor_SMD:L_Taiyo-Yuden_NR-20xx" H 6350 3350 50  0001 C CNN
+F 3 "https://www.yuden.co.jp/productdata/catalog/wound04_e.pdf" H 6350 3350 50  0001 C CNN
+F 4 "587-3452-1-ND" V 6350 3350 50  0001 C CNN "Digi-Key Part Number"
+F 5 "Taiyo Yuden" V 6350 3350 50  0001 C CNN "Manufacturer"
+F 6 "NRS2012T4R7MGJ" V 6350 3350 50  0001 C CNN "Manufacturer Part Number"
+F 7 "FIXED IND 4.7UH 910MA 241MOHM SM" V 6350 3350 50  0001 C CNN "Description"
+	1    6350 3350
+	0    -1   -1   0
+$EndComp
+$Comp
+L Device:R R3
+U 1 1 601746B0
+P 6000 3550
+F 0 "R3" H 6070 3596 50  0000 L CNN
+F 1 "400 0603" H 6070 3505 50  0000 L CNN
+F 2 "Resistor_SMD:R_0603_1608Metric" V 5930 3550 50  0001 C CNN
+F 3 "~" H 6000 3550 50  0001 C CNN
+	1    6000 3550
+	1    0    0    -1
+$EndComp
+Wire Wire Line
+	5350 3350 6000 3350
+Wire Wire Line
+	6500 3350 6700 3350
+Wire Wire Line
+	6000 3350 6000 3400
+Connection ~ 6000 3350
+Wire Wire Line
+	6000 3350 6200 3350
+Wire Wire Line
+	6000 3700 6000 3750
+Wire Wire Line
+	6000 3750 6350 3750
+Wire Wire Line
+	6350 3750 6350 3500
+Wire Wire Line
+	6350 3500 6700 3500
+Connection ~ 6000 3750
+Wire Wire Line
+	6000 3750 6000 3800
 $Comp
 L power:GND #PWR02
@@
 	1    0    0    -1
 $EndComp
+Wire Wire Line
+	5650 4250 6000 4250
+Wire Wire Line
+	6000 4250 6000 4100
+Wire Wire Line
+	5650 4250 5350 4250
+Wire Wire Line
+	5350 4250 5350 3650
 Connection ~ 5650 4250
 $Comp
@@
 	5200 3650 5200 3550
 Wire Wire Line
+	5200 3350 5350 3350
+Connection ~ 5350 3350
+Wire Wire Line
 	4850 3550 5200 3550
 Connection ~ 5200 3550
@@
 Wire Wire Line
 	5000 3350 5000 3800
+Wire Wire Line
+	5000 4250 5350 4250
+Connection ~ 5350 4250
+NoConn ~ 8000 3500
+Wire Wire Line
+	8000 3350 8450 3350
 Text HLabel 5200 3350 1    50   Input ~ 0
 V_BAT
 Wire Wire Line
+	6000 4250 6550 4250
+Wire Wire Line
+	8050 3650 8050 4250
+Connection ~ 6000 4250
+Wire Wire Line
+	8050 4250 8450 4250
+Wire Wire Line
+	8450 3650 8450 4250
+Connection ~ 8050 4250
+Wire Wire Line
+	6700 3650 6550 3650
+Wire Wire Line
+	6550 3650 6550 4250
+Connection ~ 6550 4250
+Wire Wire Line
+	6550 4250 8050 4250
+Wire Wire Line
 	3050 3350 3950 3350
-Connection ~ 5000 4250
 $Comp
 L Device:R R6
@@
 Wire Wire Line
 	5000 4100 5000 4250
-Wire Wire Line
-	3050 4250 5000 4250
-$Comp
-L HH_TexasInstruments:TPS6031x T1
-U 1 1 60B47905
-P 7250 3600
-F 0 "T1" H 7250 4115 50  0000 C CNN
-F 1 "TPS6031x" H 7250 4024 50  0000 C CNN
-F 2 "Package_SO:MSOP-10_3x3mm_P0.5mm" H 7250 3600 50  0001 C CNN
-F 3 "https://www.ti.com/general/docs/suppproductinfo.tsp?distId=10&gotoUrl=https%3A%2F%2Fwww.ti.com%2Flit%2Fgpn%2Ftps60310" H 7250 3600 50  0001 C CNN
-F 4 "296-13417-1-ND" H 7250 3600 50  0001 C CNN "Digi-Key Part Number"
-F 5 "Texas Instruments" H 7250 3600 50  0001 C CNN "Manufacturer"
-F 6 "TPS60313DGSR" H 7250 3600 50  0001 C CNN "Manufacturer Part Number"
-F 7 "IC REG CHRG PUMP 2VIN/3V 10VSSOP" H 7250 3600 50  0001 C CNN "Description"
-	1    7250 3600
-	1    0    0    -1
-$EndComp
-$Comp
-L Device:C C3
-U 1 1 60B48CDE
-P 8300 3300
-F 0 "C3" H 8415 3346 50  0000 L CNN
-F 1 "1µF X7R 0603" H 8415 3255 50  0000 L CNN
-F 2 "Capacitor_SMD:C_0603_1608Metric" H 8338 3150 50  0001 C CNN
-F 3 "~" H 8300 3300 50  0001 C CNN
-	1    8300 3300
-	1    0    0    -1
-$EndComp
-$Comp
-L Device:C C4
-U 1 1 60B4C1B9
-P 8300 3800
-F 0 "C4" H 8415 3846 50  0000 L CNN
-F 1 "1µF X7R 0603" H 8415 3755 50  0000 L CNN
-F 2 "Capacitor_SMD:C_0603_1608Metric" H 8338 3650 50  0001 C CNN
-F 3 "~" H 8300 3800 50  0001 C CNN
-	1    8300 3800
-	1    0    0    -1
-$EndComp
-Wire Wire Line
-	7950 3600 8150 3600
-Wire Wire Line
-	8150 3600 8150 3650
-Wire Wire Line
-	8150 3650 8300 3650
-Wire Wire Line
-	7950 3500 8150 3500
-Wire Wire Line
-	8150 3500 8150 3450
-Wire Wire Line
-	8150 3450 8300 3450
-Wire Wire Line
-	7950 3400 8150 3400
-Wire Wire Line
-	8150 3400 8150 3150
-Wire Wire Line
-	8150 3150 8300 3150
-Wire Wire Line
-	7950 3700 8150 3700
-Wire Wire Line
-	8150 3700 8150 3950
-Wire Wire Line
-	8150 3950 8300 3950
-NoConn ~ 7950 3850
-NoConn ~ 6550 3750
-Wire Wire Line
-	6550 3850 6350 3850
-Wire Wire Line
-	6350 3850 6350 4250
-Wire Wire Line
-	5650 4250 5850 4250
-Wire Wire Line
-	5000 4250 5650 4250
-Wire Wire Line
-	6350 3350 6350 3550
-Wire Wire Line
-	6350 3550 6550 3550
-Wire Wire Line
-	5850 3650 5850 4250
-Connection ~ 5850 4250
-Wire Wire Line
-	5850 4250 6350 4250
-Wire Wire Line
-	5200 3350 5850 3350
-$Comp
-L Device:C C2
-U 1 1 60B54C95
-P 5850 3500
-F 0 "C2" H 5965 3546 50  0000 L CNN
-F 1 "1µF X7R 0603" H 5965 3455 50  0000 L CNN
-F 2 "Capacitor_SMD:C_0603_1608Metric" H 5888 3350 50  0001 C CNN
-F 3 "~" H 5850 3500 50  0001 C CNN
-	1    5850 3500
-	1    0    0    -1
-$EndComp
-Connection ~ 5850 3350
-Wire Wire Line
-	5850 3350 6350 3350
-Text HLabel 6550 3050 0    50   Input ~ 0
-~SNOOZE
-$Comp
-L Device:R R3
-U 1 1 60BA08BD
-P 6550 2650
-F 0 "R3" H 6620 2696 50  0000 L CNN
-F 1 "100k 0603" H 6620 2605 50  0000 L CNN
-F 2 "Resistor_SMD:R_0603_1608Metric" V 6480 2650 50  0001 C CNN
-F 3 "~" H 6550 2650 50  0001 C CNN
-	1    6550 2650
-	-1   0    0    1
-$EndComp
-Wire Wire Line
-	6550 3400 6550 2800
-$Comp
-L power:GND #PWR011
-U 1 1 60BA1E65
-P 6550 2250
-F 0 "#PWR011" H 6550 2000 50  0001 C CNN
-F 1 "GND" H 6555 2077 50  0000 C CNN
-F 2 "" H 6550 2250 50  0001 C CNN
-F 3 "" H 6550 2250 50  0001 C CNN
-	1    6550 2250
-	-1   0    0    1
-$EndComp
-Wire Wire Line
-	6550 2250 6550 2500
+$Comp
+L Device:Fuse F1
+U 1 1 613D2A36
+P 3900 4250
+F 0 "F1" V 3703 4250 50  0000 C CNN
+F 1 "Fuse" V 3794 4250 50  0000 C CNN
+F 2 "Fuse:Fuse_0603_1608Metric" V 3830 4250 50  0001 C CNN
+F 3 "https://datasheets.avx.com/AccuGuardLC_0402.pdf" H 3900 4250 50  0001 C CNN
+F 4 "478-6871-1-ND" V 3900 4250 50  0001 C CNN "Digi-Key Part Number"
+F 5 "AVX Corporation" V 3900 4250 50  0001 C CNN "Manufacturer"
+F 6 "F0603G0R05FNTR" V 3900 4250 50  0001 C CNN "Manufacturer Part Number"
+F 7 "FUSE BOARD MOUNT 50MA 32VDC 0603" V 3900 4250 50  0001 C CNN "Description"
+	1    3900 4250
+	0    1    1    0
+$EndComp
+Wire Wire Line
+	3750 4250 3050 4250
+Wire Wire Line
+	4050 4250 5000 4250
+Connection ~ 5000 4250
 $EndSCHEMATC
