File: kicad/sensor-node-bl651/mcu.sch (KiCad schematic (older format))
At the start: 14 parts, among them U1 DMP2008UFG-7, Y1 32.768 kHz

Commit message: remove memsic sensors
Connections:
- net INT_M_XL: no longer names the net of BL1.10 (P0.16)
- no-connect marks 18 -> 19
Changed lines of the file:
@@
 	1    0    0    -1
 $EndComp
-Text HLabel 6600 3050 2    50   Input ~ 0
-INT_M_XL
 NoConn ~ 4800 3350
 $Comp
@@
 	8650 6250 8300 6250
 Connection ~ 8300 6250
+NoConn ~ 6600 3050
 $EndSCHEMATC
